Commit message: added anymal-d urdf and meshes

File: urdf_models/anymal/anymal.urdf (robot description, URDF)
Before this commit: robot anymal, 78 links, 77 joints
Links:
- removed link LF_HAA
- removed link LF_HFE
- removed link LF_KFE
- removed link LH_HAA
- removed link LH_HFE
- removed link LH_KFE
- removed link RF_HAA
- removed link RF_HFE
- removed link RF_KFE
- removed link RH_HAA
- removed link RH_HFE
- removed link RH_KFE
- removed link depth_camera_front_camera
- removed link depth_camera_front_camera_parent
- removed link depth_camera_front_color_frame
- removed link depth_camera_front_color_optical_frame
- removed link depth_camera_front_depth_optical_frame
- removed link depth_camera_left_color_frame
- removed link depth_camera_left_color_optical_frame
- removed link depth_camera_rear_camera
- removed link depth_camera_rear_camera_parent
- removed link depth_camera_rear_color_frame
- removed link depth_camera_rear_color_optical_frame
- removed link depth_camera_rear_depth_optical_frame
- removed link depth_camera_right_color_frame
- removed link depth_camera_right_color_optical_frame
- removed link docking_hatch_cover
- removed link handle
- removed link hatch
- removed link lidar_cage
- removed link remote
- added link LF_HAA_drive, mass 2.01511; visual mesh filename=package://anymal_d_simple_description/meshes/drive.dae scale=1.0 1.0 1.0
- added link LF_HFE_drive, mass 2.01511; collision cylinder length=0.119 radius=0.05375; visual mesh filename=package://anymal_d_simple_description/meshes/drive.dae scale=1.0 1.0 1.0
- added link LF_HFE_output, mass 0.001
- added link LF_KFE_drive, mass 2.01511; collision cylinder length=0.119 radius=0.05375; visual mesh filename=package://anymal_d_simple_description/meshes/drive.dae scale=1.0 1.0 1.0
- added link LH_HAA_drive, mass 2.01511; visual mesh filename=package://anymal_d_simple_description/meshes/drive.dae scale=1.0 1.0 1.0
- added link LH_HFE_drive, mass 2.01511; collision cylinder length=0.119 radius=0.05375; visual mesh filename=package://anymal_d_simple_description/meshes/drive.dae scale=1.0 1.0 1.0
- added link LH_HFE_output, mass 0.001
- added link LH_KFE_drive, mass 2.01511; collision cylinder length=0.119 radius=0.05375; visual mesh filename=package://anymal_d_simple_description/meshes/drive.dae scale=1.0 1.0 1.0
- added link RF_HAA_drive, mass 2.01511; visual mesh filename=package://anymal_d_simple_description/meshes/drive.dae scale=1.0 1.0 1.0
- added link RF_HFE_drive, mass 2.01511; collision cylinder length=0.119 radius=0.05375; visual mesh filename=package://anymal_d_simple_description/meshes/drive.dae scale=1.0 1.0 1.0
- added link RF_HFE_output, mass 0.001
- added link RF_KFE_drive, mass 2.01511; collision cylinder length=0.119 radius=0.05375; visual mesh filename=package://anymal_d_simple_description/meshes/drive.dae scale=1.0 1.0 1.0
- added link RH_HAA_drive, mass 2.01511; visual mesh filename=package://anymal_d_simple_description/meshes/drive.dae scale=1.0 1.0 1.0
- added link RH_HFE_drive, mass 2.01511; collision cylinder length=0.119 radius=0.05375; visual mesh filename=package://anymal_d_simple_description/meshes/drive.dae scale=1.0 1.0 1.0
- added link RH_HFE_output, mass 0.001
- added link RH_KFE_drive, mass 2.01511; collision cylinder length=0.119 radius=0.05375; visual mesh filename=package://anymal_d_simple_description/meshes/drive.dae scale=1.0 1.0 1.0
- added link body_top
- added link depth_camera_front_lower_camera, mass 0.06355
- added link depth_camera_front_lower_camera_parent
- added link depth_camera_front_lower_depth_frame
- added link depth_camera_front_lower_depth_optical_frame
- added link depth_camera_front_upper_camera, mass 0.06355
- added link depth_camera_front_upper_camera_parent
- added link depth_camera_front_upper_depth_frame
- added link depth_camera_front_upper_depth_optical_frame
- added link depth_camera_left_depth_frame
- added link depth_camera_rear_lower_camera, mass 0.06355
- added link depth_camera_rear_lower_camera_parent
- added link depth_camera_rear_lower_depth_frame
- added link depth_camera_rear_lower_depth_optical_frame
- added link depth_camera_rear_upper_camera, mass 0.06355
- added link depth_camera_rear_upper_camera_parent
- added link depth_camera_rear_upper_depth_frame
- added link depth_camera_rear_upper_depth_optical_frame
- added link depth_camera_right_depth_frame
- added link docking_socket, mass 0.21905; visual mesh filename=package://anymal_d_simple_description/meshes/docking_socket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 scale=1.0 1.0 1.0
- added link face_shell_front, mass 0.1369; visual mesh filename=package://anymal_d_simple_description/meshes/face_shell.dae scale=1.0 1.0 1.0
- added link face_shell_rear, mass 0.1369; visual mesh filename=package://anymal_d_simple_description/meshes/face_shell.dae scale=1.0 1.0 1.0
- added link hbc_receiver, mass 0.60727
- added link inspection_payload_camera
- added link inspection_payload_camera_default
- added link inspection_payload_head
- added link inspection_payload_light
- added link inspection_payload_microphone
- added link inspection_payload_mount, mass 0.21580; collision box size=0.16 0.135 0.015; visual mesh filename=package://anymal_d_simple_description/meshes/mount.dae scale=1 1 1
- added link inspection_payload_pan, mass 3.18886; collision box size=0.18 0.24 0.21; visual mesh filename=package://anymal_d_simple_description/meshes/pan.dae scale=1 1 1
- added link inspection_payload_thermal_camera
- added link inspection_payload_tilt, mass 2.084; visual mesh filename=package://anymal_d_simple_description/meshes/tilt.dae scale=1 1 1
- added link lidar_parent
- link LF_FOOT: mass 0.25 -> 0.29644; geometry collision cylinder length=0.39572 radius=0.0175; collision sphere radius=0.031455
- link LF_hip_fixed: mass 0.74 -> 0.36386; geometry visual mesh filename=package://anymal_d_simple_description/meshes/hip.dae scale=1.0 1.0 1.0
- link LF_shank_fixed: mass 0.33742 -> 0.49854; geometry collision box size=0.13283 0.08302 0.05732; collision cylinder length=0.05732 radius=0.071
- link LF_thigh_fixed: mass 1.03 -> 1.10098; geometry collision box size=0.093 0.063 0.285; collision cylinder length=0.08313000000000001 radius=0.07
- link LH_FOOT: mass 0.25 -> 0.29644; geometry collision cylinder length=0.39572 radius=0.0175; collision sphere radius=0.031455
- link LH_hip_fixed: mass 0.74 -> 0.36386; geometry visual mesh filename=package://anymal_d_simple_description/meshes/hip.dae scale=1.0 1.0 1.0
- link LH_shank_fixed: mass 0.33742 -> 0.49854; geometry collision box size=0.13283 0.08302 0.05732; collision cylinder length=0.05732 radius=0.071
- link LH_thigh_fixed: mass 1.03 -> 1.10098; geometry collision box size=0.093 0.063 0.285; collision cylinder length=0.08313000000000001 radius=0.07
- link RF_FOOT: mass 0.25 -> 0.29644; geometry collision cylinder length=0.39572 radius=0.0175; collision sphere radius=0.031455
- link RF_hip_fixed: mass 0.74 -> 0.36386; geometry visual mesh filename=package://anymal_d_simple_description/meshes/hip.dae scale=1.0 1.0 1.0
- link RF_shank_fixed: mass 0.33742 -> 0.49854; geometry collision box size=0.13283 0.08302 0.05732; collision cylinder length=0.05732 radius=0.071
- link RF_thigh_fixed: mass 1.03 -> 1.10098; geometry collision box size=0.093 0.063 0.285; collision cylinder length=0.08313000000000001 radius=0.07
- link RH_FOOT: mass 0.25 -> 0.29644; geometry collision cylinder length=0.39572 radius=0.0175; collision sphere radius=0.031455
- link RH_hip_fixed: mass 0.74 -> 0.36386; geometry visual mesh filename=package://anymal_d_simple_description/meshes/hip.dae scale=1.0 1.0 1.0
- link RH_shank_fixed: mass 0.33742 -> 0.49854; geometry collision box size=0.13283 0.08302 0.05732; collision cylinder length=0.05732 radius=0.071
- link RH_thigh_fixed: mass 1.03 -> 1.10098; geometry collision box size=0.093 0.063 0.285; collision cylinder length=0.08313000000000001 radius=0.07
- link base: geometry collision box size=0.894 0.1615 0.256; collision cylinder length=0.1482 radius=0.089
- link base_inertia: mass 6.222 -> 8.27629
- link battery: mass 5.53425 -> 5.51206; geometry visual mesh filename=package://anymal_d_simple_description/meshes/battery.dae scale=1.0 1.0 1.0
- link bottom_shell: mass 1.15 -> 0.73783; geometry visual mesh filename=package://anymal_d_simple_description/meshes/bottom_shell.d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 scale=1.0 1.0 1.0
- link depth_camera_left_camera: mass 0.16043 -> 0.11196; geometry 
- link depth_camera_right_camera: mass 0.16043 -> 0.11196; geometry 
- link face_front: mass 0.73 -> 0.48634; geometry 
- link face_rear: mass 0.73 -> 0.48634; geometry 
- link imu_link: mass 0.01 -> None; geometry 
- link lidar: mass 0.695 -> 0.9017; geometry collision cylinder length=0.1355 radius=0.07; visual mesh filename=package://anymal_d_simple_description/meshes/lidar.dae
- link top_shell: mass 0.534 -> 0.32381; geometry visual mesh filename=package://anymal_d_simple_description/meshes/top_shell.dae scale=1.0 1.0 1.0
- link wide_angle_camera_front_camera: mass 0.287 -> None; geometry 
- link wide_angle_camera_rear_camera: mass 0.287 -> None; geometry 
Joints:
- removed joint LF_THIGH_LF_thigh_fixed
- removed joint LF_hip_fixed_LF_HFE
- removed joint LF_thigh_fixed_LF_KFE
- removed joint LH_THIGH_LH_thigh_fixed
- removed joint LH_hip_fixed_LH_HFE
- removed joint LH_thigh_fixed_LH_KFE
- removed joint RF_THIGH_RF_thigh_fixed
- removed joint RF_hip_fixed_RF_HFE
- removed joint RF_thigh_fixed_RF_KFE
- removed joint RH_THIGH_RH_thigh_fixed
- removed joint RH_hip_fixed_RH_HFE
- removed joint RH_thigh_fixed_RH_KFE
- removed joint base_LF_HAA
- removed joint base_LH_HAA
- removed joint base_RF_HAA
- removed joint base_RH_HAA
- removed joint base_handle
- removed joint base_hatch
- removed joint base_remote
- removed joint base_to_docking_hatch_cover
- removed joint base_to_lidar_cage
- removed joint depth_camera_front_camera_parent_to_color_frame
- removed joint depth_camera_front_camera_parent_to_depth_optical_frame
- removed joint depth_camera_front_camera_to_camera_parent
- removed joint depth_camera_front_color_frame_to_color_optical_frame
- removed joint depth_camera_left_camera_parent_to_color_frame
- removed joint depth_camera_left_camera_parent_to_depth_optical_frame
- removed joint depth_camera_left_color_frame_to_color_optical_frame
- removed joint depth_camera_rear_camera_parent_to_color_frame
- removed joint depth_camera_rear_camera_parent_to_depth_optical_frame
- removed joint depth_camera_rear_camera_to_camera_parent
- removed joint depth_camera_rear_color_frame_to_color_optical_frame
- removed joint depth_camera_right_camera_parent_to_color_frame
- removed joint depth_camera_right_camera_parent_to_depth_optical_frame
- removed joint depth_camera_right_color_frame_to_color_optical_frame
- removed joint face_front_to_depth_camera_front_camera
- removed joint face_rear_to_depth_camera_rear_camera
- removed joint lidar_cage_to_lidar
- added joint LF_HFE_drive_LF_thigh_fixed: type fixed, parent LF_HFE_drive, child LF_thigh_fixed, origin xyz=0 0 0 rpy=0 0 1.5707963267948966
- added joint LF_THIGH_to_LF_HFE_drive: type fixed, parent LF_THIGH, child LF_HFE_drive, origin xyz=0 0 0 rpy=0 0 0
- added joint LF_hip_fixed_LF_HFE_output: type fixed, parent LF_hip_fixed, child LF_HFE_output, origin xyz=0.069 0.006 0.0 rpy=0 0 -1.5707963267948966
- added joint LF_thigh_fixed_LF_KFE_drive: type fixed, parent LF_thigh_fixed, child LF_KFE_drive, origin xyz=0.0 0.1805 -0.285 rpy=0 0 1.5707963267948966
- added joint LH_HFE_drive_LH_thigh_fixed: type fixed, parent LH_HFE_drive, child LH_thigh_fixed, origin xyz=0 0 0 rpy=0 0 1.5707963267948966
- added joint LH_THIGH_to_LH_HFE_drive: type fixed, parent LH_THIGH, child LH_HFE_drive, origin xyz=0 0 0 rpy=0 0 0
- added joint LH_hip_fixed_LH_HFE_output: type fixed, parent LH_hip_fixed, child LH_HFE_output, origin xyz=-0.069 0.006 0.0 rpy=0 0 -1.5707963267948966
- added joint LH_thigh_fixed_LH_KFE_drive: type fixed, parent LH_thigh_fixed, child LH_KFE_drive, origin xyz=-0.0 0.1805 -0.285 rpy=0 0 1.5707963267948966
- added joint RF_HFE_drive_RF_thigh_fixed: type fixed, parent RF_HFE_drive, child RF_thigh_fixed, origin xyz=0 0 0 rpy=0 0 -1.5707963267948966
- added joint RF_THIGH_to_RF_HFE_drive: type fixed, parent RF_THIGH, child RF_HFE_drive, origin xyz=0 0 0 rpy=0 0 0
- added joint RF_hip_fixed_RF_HFE_output: type fixed, parent RF_hip_fixed, child RF_HFE_output, origin xyz=0.069 -0.006 0.0 rpy=0 0 1.5707963267948966
- added joint RF_thigh_fixed_RF_KFE_drive: type fixed, parent RF_thigh_fixed, child RF_KFE_drive, origin xyz=0.0 -0.1805 -0.285 rpy=0 0 -1.5707963267948966
- added joint RH_HFE_drive_RH_thigh_fixed: type fixed, parent RH_HFE_drive, child RH_thigh_fixed, origin xyz=0 0 0 rpy=0 0 -1.5707963267948966
- added joint RH_THIGH_to_RH_HFE_drive: type fixed, parent RH_THIGH, child RH_HFE_drive, origin xyz=0 0 0 rpy=0 0 0
- added joint RH_hip_fixed_RH_HFE_output: type fixed, parent RH_hip_fixed, child RH_HFE_output, origin xyz=-0.069 -0.006 0.0 rpy=0 0 1.5707963267948966
- added joint RH_thigh_fixed_RH_KFE_drive: type fixed, parent RH_thigh_fixed, child RH_KFE_drive, origin xyz=-0.0 -0.1805 -0.285 rpy=0 0 -1.5707963267948966
- added joint base_LF_HAA_drive: type fixed, parent base, child LF_HAA_drive, origin xyz=0.304 0.109 0.0 rpy=0 0 0.0
- added joint base_LH_HAA_drive: type fixed, parent base, child LH_HAA_drive, origin xyz=-0.304 0.109 0.0 rpy=0 0 -3.141592653589793
- added joint base_RF_HAA_drive: type fixed, parent base, child RF_HAA_drive, origin xyz=0.304 -0.109 0.0 rpy=0 0 0.0
- added joint base_RH_HAA_drive: type fixed, parent base, child RH_HAA_drive, origin xyz=-0.304 -0.109 0.0 rpy=0 0 -3.141592653589793
- added joint base_face_shell_front: type fixed, parent face_front, child face_shell_front, origin xyz=0 0 0 rpy=0 0 0
- added joint base_face_shell_rear: type fixed, parent face_rear, child face_shell_rear, origin xyz=0 0 0 rpy=0 0 0
- added joint base_hbc_receiver: type fixed, parent base, child hbc_receiver, origin xyz=-0.04350 0.0 0.14400 rpy=0 0 0
- added joint base_to_body_top: type fixed, parent base, child body_top, origin xyz=0 0 0.144 rpy=0 0 0
- added joint base_to_docking_socket: type fixed, parent base, child docking_socket, origin xyz=0.26132 0.0 -0.06205 rpy=0 0 0
- added joint base_to_inspection_payload_mount: type fixed, parent base, child inspection_payload_mount, origin xyz=0.14253 0.0 0.092 rpy=0 0 0
- added joint base_to_lidar_parent: type fixed, parent base, child lidar_parent, origin xyz=-0.310 0.0 0.1585 rpy=0 0 1.5707963267948966
- added joint depth_camera_front_lower_camera_depth_to_depth_optical_frame: type fixed, parent depth_camera_front_lower_depth_frame, child depth_camera_front_lower_depth_optical_frame, origin xyz=0.0 0.0 0.0 rpy=-1.5707963267948966 0.0 -1.5707963267948966
- added joint depth_camera_front_lower_camera_parent_to_depth_frame: type fixed, parent depth_camera_front_lower_camera_parent, child depth_camera_front_lower_depth_frame, origin xyz=0.0 0.0 0.0 rpy=0.0 0.0 0.0
- added joint depth_camera_front_lower_camera_to_camera_parent: type fixed, parent depth_camera_front_lower_camera, child depth_camera_front_lower_camera_parent, origin xyz=0.0 0.0 0.0 rpy=3.141592653589793 0.0 0.0
- added joint depth_camera_front_upper_camera_depth_to_depth_optical_frame: type fixed, parent depth_camera_front_upper_depth_frame, child depth_camera_front_upper_depth_optical_frame, origin xyz=0.0 0.0 0.0 rpy=-1.5707963267948966 0.0 -1.5707963267948966
- added joint depth_camera_front_upper_camera_parent_to_depth_frame: type fixed, parent depth_camera_front_upper_camera_parent, child depth_camera_front_upper_depth_frame, origin xyz=0.0 0.0 0.0 rpy=0.0 0.0 0.0
- added joint depth_camera_front_upper_camera_to_camera_parent: type fixed, parent depth_camera_front_upper_camera, child depth_camera_front_upper_camera_parent, origin xyz=0.0 0.0 0.0 rpy=3.141592653589793 0.0 0.0
- added joint depth_camera_left_camera_depth_to_depth_optical_frame: type fixed, parent depth_camera_left_depth_frame, child depth_camera_left_depth_optical_frame, origin xyz=0.0 0.0 0.0 rpy=-1.5707963267948966 0.0 -1.5707963267948966
- added joint depth_camera_left_camera_parent_to_depth_frame: type fixed, parent depth_camera_left_camera_parent, child depth_camera_left_depth_frame, origin xyz=0.0 0.0 0.0 rpy=0.0 0.0 0.0
- added joint depth_camera_rear_lower_camera_depth_to_depth_optical_frame: type fixed, parent depth_camera_rear_lower_depth_frame, child depth_camera_rear_lower_depth_optical_frame, origin xyz=0.0 0.0 0.0 rpy=-1.5707963267948966 0.0 -1.5707963267948966
- added joint depth_camera_rear_lower_camera_parent_to_depth_frame: type fixed, parent depth_camera_rear_lower_camera_parent, child depth_camera_rear_lower_depth_frame, origin xyz=0.0 0.0 0.0 rpy=0.0 0.0 0.0
- added joint depth_camera_rear_lower_camera_to_camera_parent: type fixed, parent depth_camera_rear_lower_camera, child depth_camera_rear_lower_camera_parent, origin xyz=0.0 0.0 0.0 rpy=3.141592653589793 0.0 0.0
- added joint depth_camera_rear_upper_camera_depth_to_depth_optical_frame: type fixed, parent depth_camera_rear_upper_depth_frame, child depth_camera_rear_upper_depth_optical_frame, origin xyz=0.0 0.0 0.0 rpy=-1.5707963267948966 0.0 -1.5707963267948966
- added joint depth_camera_rear_upper_camera_parent_to_depth_frame: type fixed, parent depth_camera_rear_upper_camera_parent, child depth_camera_rear_upper_depth_frame, origin xyz=0.0 0.0 0.0 rpy=0.0 0.0 0.0
- added joint depth_camera_rear_upper_camera_to_camera_parent: type fixed, parent depth_camera_rear_upper_camera, child depth_camera_rear_upper_camera_parent, origin xyz=0.0 0.0 0.0 rpy=3.141592653589793 0.0 0.0
- added joint depth_camera_right_camera_depth_to_depth_optical_frame: type fixed, parent depth_camera_right_depth_frame, child depth_camera_right_depth_optical_frame, origin xyz=0.0 0.0 0.0 rpy=-1.5707963267948966 0.0 -1.5707963267948966
- added joint depth_camera_right_camera_parent_to_depth_frame: type fixed, parent depth_camera_right_camera_parent, child depth_camera_right_depth_frame, origin xyz=0.0 0.0 0.0 rpy=0.0 0.0 0.0
- added joint face_front_to_depth_camera_front_lower_camera: type fixed, parent face_front, child depth_camera_front_lower_camera, origin xyz=-0.04028 -0.025 -0.08051 rpy=0.0 1.0471975511965976 0
- added joint face_front_to_depth_camera_front_upper_camera: type fixed, parent face_front, child depth_camera_front_upper_camera, origin xyz=-0.00993 -0.025 -0.04096 rpy=0.0 0.2617993877991494 0
- added joint face_rear_to_depth_camera_rear_lower_camera: type fixed, parent face_rear, child depth_camera_rear_lower_camera, origin xyz=-0.04028 -0.025 -0.08051 rpy=0.0 1.0471975511965976 0
- added joint face_rear_to_depth_camera_rear_upper_camera: type fixed, parent face_rear, child depth_camera_rear_upper_camera, origin xyz=-0.00993 -0.025 -0.04096 rpy=0.0 0.2617993877991494 0
- added joint inspection_payload_head_to_camera: type fixed, parent inspection_payload_head, child inspection_payload_camera, origin xyz=0.055 -0.023 0.031 rpy=-1.57079633 0 -1.57079633
- added joint inspection_payload_head_to_light: type fixed, parent inspection_payload_head, child inspection_payload_light, origin xyz=0.05495 0.03000 0.03116 rpy=-1.57079633 0 -1.57079633
- added joint inspection_payload_head_to_microphone: type fixed, parent inspection_payload_head, child inspection_payload_microphone, origin xyz=0.06840 0.02300 -0.03000 rpy=-1.57079633 0 -1.57079633
- added joint inspection_payload_head_to_thermal_camera: type fixed, parent inspection_payload_head, child inspection_payload_thermal_camera, origin xyz=0.06840 -0.02300 -0.03000 rpy=-1.57079633 0 -1.57079633
- added joint inspection_payload_mount_to_camera_default: type fixed, parent inspection_payload_mount, child inspection_payload_camera_default, origin xyz=0.0 0.0 0.175 rpy=0 0 0
- added joint inspection_payload_mount_to_pan: type revolute, parent inspection_payload_mount, child inspection_payload_pan, origin xyz=0 0 0.023 rpy=0 0 0, axis 0 0 1, limit lower=-2.6 upper=2.6 effort=20 velocity=2
- added joint inspection_payload_pan_to_tilt: type revolute, parent inspection_payload_pan, child inspection_payload_tilt, origin xyz=0.03 0 0.152 rpy=0 0 0, axis 0 1 0, limit lower=-1.570796 upper=1.570796 effort=20 velocity=2
- added joint inspection_payload_tilt_to_head: type fixed, parent inspection_payload_tilt, child inspection_payload_head, origin xyz=0.0 0.0 0.0 rpy=0 0 0
- added joint lidar_parent_to_lidar: type fixed, parent lidar_parent, child lidar, origin xyz=0 0 0 rpy=0 0 1.5707963267948966
- joint LF_HAA: limit lower=-0.72 upper=0.49 effort=80.0 velocity=7.5 -> lower=-0.7853985 upper=0.6108655 effort=80.0 velocity=8.5; parent LF_HAA -> LF_HAA_drive
- joint LF_HFE: axis 1 0 0 -> -1 0 0; limit lower=-9.42477796077 upper=9.42477796077 effort=80.0 velocity=7.5 -> lower=-9.42477796076938 upper=9.42477796076938 effort=80.0 velocity=8.5; parent LF_HFE -> LF_HFE_output
- joint LF_HIP_LF_hip_fixed: origin xyz=0 0 0 rpy=-2.61799387799 0 0.0 -> xyz=0 0 0 rpy=0 0 0.0
- joint LF_KFE: limit lower=-9.42477796077 upper=9.42477796077 effort=80.0 velocity=7.5 -> lower=-9.42477796076938 upper=9.42477796076938 effort=80.0 velocity=8.5; parent LF_KFE -> LF_KFE_drive
- joint LF_shank_LF_shank_fixed: origin xyz=0 0 0 rpy=0 0 -1.57079632679 -> xyz=0 0 0 rpy=0 0 -1.5707963267948966
- joint LF_shank_fixed_LF_FOOT: origin xyz=0.08795 0.01305 -0.33797 rpy=0 0 0 -> xyz=0.1 0.02225 -0.39246 rpy=0 0 0
- joint LH_HAA: limit lower=-0.72 upper=0.49 effort=80.0 velocity=7.5 -> lower=-0.7853985 upper=0.6108655 effort=80.0 velocity=8.5; parent LH_HAA -> LH_HAA_drive
- joint LH_HFE: axis 1 0 0 -> -1 0 0; limit lower=-9.42477796077 upper=9.42477796077 effort=80.0 velocity=7.5 -> lower=-9.42477796076938 upper=9.42477796076938 effort=80.0 velocity=8.5; parent LH_HFE -> LH_HFE_output
- joint LH_HIP_LH_hip_fixed: origin xyz=0 0 0 rpy=-2.61799387799 0 -3.14159265359 -> xyz=0 0 0 rpy=0 0 -3.141592653589793
- joint LH_KFE: limit lower=-9.42477796077 upper=9.42477796077 effort=80.0 velocity=7.5 -> lower=-9.42477796076938 upper=9.42477796076938 effort=80.0 velocity=8.5; parent LH_KFE -> LH_KFE_drive
- joint LH_shank_LH_shank_fixed: origin xyz=0 0 0 rpy=0 0 -1.57079632679 -> xyz=0 0 0 rpy=0 0 -1.5707963267948966
- joint LH_shank_fixed_LH_FOOT: origin xyz=-0.08795 0.01305 -0.33797 rpy=0 0 0 -> xyz=-0.1 0.02225 -0.39246 rpy=0 0 0
- joint RF_HAA: limit lower=-0.49 upper=0.72 effort=80.0 velocity=7.5 -> lower=-0.6108655 upper=0.7853985 effort=80.0 velocity=8.5; parent RF_HAA -> RF_HAA_drive
- joint RF_HFE: axis -1 0 0 -> 1 0 0; limit lower=-9.42477796077 upper=9.42477796077 effort=80.0 velocity=7.5 -> lower=-9.42477796076938 upper=9.42477796076938 effort=80.0 velocity=8.5; parent RF_HFE -> RF_HFE_output
- joint RF_HIP_RF_hip_fixed: origin xyz=0 0 0 rpy=2.61799387799 0 0.0 -> xyz=0 0 0 rpy=0 0 0.0
- joint RF_KFE: limit lower=-9.42477796077 upper=9.42477796077 effort=80.0 velocity=7.5 -> lower=-9.42477796076938 upper=9.42477796076938 effort=80.0 velocity=8.5; parent RF_KFE -> RF_KFE_drive
- joint RF_shank_RF_shank_fixed: origin xyz=0 0 0 rpy=0 0 1.57079632679 -> xyz=0 0 0 rpy=0 0 1.5707963267948966
- joint RF_shank_fixed_RF_FOOT: origin xyz=0.08795 -0.01305 -0.33797 rpy=0 0 0 -> xyz=0.1 -0.02225 -0.39246 rpy=0 0 0
- joint RH_HAA: limit lower=-0.49 upper=0.72 effort=80.0 velocity=7.5 -> lower=-0.6108655 upper=0.7853985 effort=80.0 velocity=8.5; parent RH_HAA -> RH_HAA_drive
- joint RH_HFE: axis -1 0 0 -> 1 0 0; limit lower=-9.42477796077 upper=9.42477796077 effort=80.0 velocity=7.5 -> lower=-9.42477796076938 upper=9.42477796076938 effort=80.0 velocity=8.5; parent RH_HFE -> RH_HFE_output
- joint RH_HIP_RH_hip_fixed: origin xyz=0 0 0 rpy=2.61799387799 0 -3.14159265359 -> xyz=0 0 0 rpy=0 0 -3.141592653589793
- joint RH_KFE: limit lower=-9.42477796077 upper=9.42477796077 effort=80.0 velocity=7.5 -> lower=-9.42477796076938 upper=9.42477796076938 effort=80.0 velocity=8.5; parent RH_KFE -> RH_KFE_drive
- joint RH_shank_RH_shank_fixed: origin xyz=0 0 0 rpy=0 0 1.57079632679 -> xyz=0 0 0 rpy=0 0 1.5707963267948966
- joint RH_shank_fixed_RH_FOOT: origin xyz=-0.08795 -0.01305 -0.33797 rpy=0 0 0 -> xyz=-0.1 -0.02225 -0.39246 rpy=0 0 0
- joint base_face_front: origin xyz=0.4145 0 0 rpy=0 0 -0.0 -> xyz=0.4087 0 0.0205 rpy=0 0 -0.0
- joint base_face_rear: origin xyz=-0.4145 0 0 rpy=0 0 3.14159265359 -> xyz=-0.4087 0 0.0205 rpy=0 0 3.141592653589793
- joint base_to_depth_camera_left_camera: origin xyz=0.0 0.07646 0.02905 rpy=0.0 0.523598775598 1.57079632679 -> xyz=-0.02500 0.09230 0.01230 rpy=0.0 0.7330382858376184 1.5707963267948966
- joint base_to_depth_camera_right_camera: origin xyz=0.0 -0.07646 0.02905 rpy=0.0 0.523598775598 -1.57079632679 -> xyz=0.02500 -0.09230 0.01230 rpy=0.0 0.7330382858376184 -1.5707963267948966
- joint depth_camera_left_camera_to_camera_parent: origin xyz=0.0255 0.0175 0.0 rpy=0.0 0.0 0.0 -> xyz=0.0 0.0 0.0 rpy=0.0 0.0 0.0
- joint depth_camera_right_camera_to_camera_parent: origin xyz=0.0255 0.0175 0.0 rpy=0.0 0.0 0.0 -> xyz=0.0 0.0 0.0 rpy=0.0 0.0 0.0
- joint face_front_to_wide_angle_camera_front_camera: origin xyz=0.09850 0.0 0.01497 rpy=0 0 0 -> xyz=0.0 0.0 0.0 rpy=0 0 0
- joint face_rear_to_wide_angle_camera_rear_camera: origin xyz=0.09850 0.0 0.01497 rpy=0 0 0 -> xyz=0.0 0.0 0.0 rpy=0 0 0
- joint imu_joint: origin xyz=0.2488 0.00835 0.04628 rpy=0.0 0.0 1.57079632679 -> xyz=-0.25565 0.00255 0.07672 rpy=3.141592653589793 0.0 3.141592653589793
- joint wide_angle_camera_front_camera_to_camera_parent: origin xyz=0.0 0.0 0.0 rpy=-1.57079632679 0.0 -1.57079632679 -> xyz=-0.00421 0.0 0.0 rpy=-1.5707963267948966 0.0 -1.5707963267948966
- joint wide_angle_camera_rear_camera_to_camera_parent: origin xyz=0.0 0.0 0.0 rpy=-1.57079632679 0.0 -1.57079632679 -> xyz=-0.00421 0.0 0.0 rpy=-1.5707963267948966 0.0 -1.5707963267948966
