Commit message: now with obj files

File: project_starter/anymal/anymal.urdf (robot description, URDF)
Before this commit: robot spot, 26 links, 25 joints
Links:
- link front_left_hip: geometry visual mesh filename=../../../urdf_models/anymal/meshes/base.obj

File: project_starter/spot/spot.urdf (robot description, URDF)
Before this commit: robot spot, 26 links, 25 joints
Links:
- link body: geometry visual mesh filename=../../../urdf_models/anymal/meshes/tilt.obj
- link rear_left_upper_leg: geometry visual mesh filename=../../../urdf_models/anymal/meshes/tilt.obj

File: urdf_models/spot/spot.urdf (robot description, URDF)
Before this commit: robot spot, 26 links, 25 joints
Links:
- link body: geometry visual mesh filename=../../../model/anymal/meshes/tilt.obj
